File: cca/lamp_rpi3_button_relay_if.kicad_pcb (KiCad board)
At the start: 2 copper layers, 41.9 x 38.1 mm, 5 parts, among them P1 lamp_cca_rpi3_conn, P2 lamp_cca_relay_conn, SW1 TSA12110

Commit message: minor cca updates
Parts:
- moved SW1 12.7 mm to (35.6, 50.8)
- moved REF** 12.7 mm to (64.1, 28.6)
- moved P1 12.7 mm to (27.9, 35.6)
- moved P2 12.7 mm to (61.0, 35.6)
Other:
- board size 41.9 x 38.1 mm -> 41.9 x 50.8 mm
Changed lines of the file:
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@@
     (links 7)
     (no_connects 0)
-    (area 25.324999 38.024999 67.385001 76.275001)
+    (area 25.14 36.652 67.385001 77.494)
     (thickness 1.6)
     (drawings 4)
@@
       (outputformat 1)
       (mirror false)
-      (drillshape 1)
+      (drillshape 0)
       (scaleselection 1)
-      (outputdirectory ""))
+      (outputdirectory fab_output.nogit/))
   )
   (net 0 "")
@@
   )
   (module Connect:1pin (layer F.Cu)
-    (at 64.135 41.275)
+    (at 64.135 28.575)
     (descr "module 1 pin (ou trou mecanique de percage)")
     (tags DEV)
@@
   )
   (module t_footprints:conn_4_big_pads (layer F.Cu)
-    (at 27.94 48.26)
+    (at 27.94 35.56)
     (fp_text reference P1 (at 0 -4) (layer F.SilkS)
       (effects (font (size 1.2 1.2) (thickness 0.15)))
@@
   )
   (module t_footprints:conn_4_big_pads (layer F.Cu)
-    (at 60.96 48.26)
+    (at 60.96 35.56)
     (fp_text reference P2 (at 0 -4) (layer F.SilkS)
       (effects (font (size 1.2 1.2) (thickness 0.15)))
@@
   )
   (module t_footprints:TSA12110 (layer F.Cu)
-    (at 35.56 63.5)
+    (at 35.56 50.8)
     (fp_text reference SW1 (at 6.25 -4.5 180) (layer F.SilkS)
       (effects (font (size 1.2 1.2) (thickness 0.15)))
@@
     (pad 1 thru_hole circle (at 0 0) (size 4.064 4.064) (drill 3.175) (layers *.Cu *.Mask F.SilkS))
   )
-  (gr_line (start 67.31 38.1) (end 25.4 38.1) (angle 90) (layer Edge.Cuts) (width 0.15))
-  (gr_line (start 67.31 76.2) (end 67.31 38.1) (angle 90) (layer Edge.Cuts) (width 0.15))
+  (gr_line (start 67.31 25.4) (end 25.4 25.4) (angle 90) (layer Edge.Cuts) (width 0.15))
+  (gr_line (start 67.31 76.2) (end 67.31 25.4) (angle 90) (layer Edge.Cuts) (width 0.15))
   (gr_line (start 25.4 76.2) (end 67.31 76.2) (angle 90) (layer Edge.Cuts) (width 0.15))
-  (gr_line (start 25.4 38.1) (end 25.4 76.2) (angle 90) (layer Edge.Cuts) (width 0.15))
-  (segment (start 35.56 63.5) (end 31.18 63.5) (width 0.8) (layer F.Cu) (net 3))
-  (segment (start 31.18 63.5) (end 27.94 60.26) (width 0.8) (layer F.Cu) (net 3))
-  (segment (start 27.94 54.26) (end 30.74 54.26) (width 0.8) (layer F.Cu) (net 4))
-  (segment (start 30.74 54.26) (end 36.74 60.26) (width 0.8) (layer F.Cu) (net 4))
-  (segment (start 36.74 60.26) (end 60.96 60.26) (width 0.8) (layer F.Cu) (net 4))
-  (segment (start 60.96 60.26) (end 58.16 60.26) (width 0.8) (layer F.Cu) (net 4))
+  (gr_line (start 25.4 25.4) (end 25.4 76.2) (angle 90) (layer Edge.Cuts) (width 0.15))
+  (segment (start 35.56 50.8) (end 31.18 50.8) (width 0.8) (layer F.Cu) (net 3))
+  (segment (start 31.18 50.8) (end 27.94 47.56) (width 0.8) (layer F.Cu) (net 3))
+  (segment (start 27.94 41.56) (end 30.74 41.56) (width 0.8) (layer F.Cu) (net 4))
+  (segment (start 30.74 41.56) (end 36.74 47.56) (width 0.8) (layer F.Cu) (net 4))
+  (segment (start 36.74 47.56) (end 60.96 47.56) (width 0.8) (layer F.Cu) (net 4))
+  (segment (start 60.96 47.56) (end 58.16 47.56) (width 0.8) (layer F.Cu) (net 4))
   (zone (net 2) (net_name GND) (layer F.Cu) (hatch edge 0.508)
     (connect_pads (clearance 1.6))
@@
     (polygon
       (pts
-        (xy 25.4 51.435) (xy 25.4 76.2) (xy 67.31 76.2) (xy 67.31 51.435)
+        (xy 25.4 38.735) (xy 25.4 63.5) (xy 67.31 63.5) (xy 67.31 38.735)
       )
     )
@@
     (polygon
       (pts
-        (xy 67.31 49.53) (xy 67.31 45.72) (xy 25.4 45.72) (xy 25.4 49.53)
+        (xy 67.31 36.83) (xy 67.31 33.02) (xy 25.4 33.02) (xy 25.4 36.83)
       )
     )
